File: remote_sch.sch (EAGLE design)
At the start: 7 parts

Commit message: a
Connections:
- net N$1: now also U$1.P0.03/AIN1@05; no longer U$1.P0.00/XL1@02
Changed lines of the file:
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@@
 <segment>
 <pinref part="POT" gate="G$1" pin="2"/>
-<pinref part="U$1" gate="U$1" pin="P0.00/XL1@02"/>
-<wire x1="12.7" y1="55.88" x2="55.88" y2="55.88" width="0.1524" layer="91"/>
+<wire x1="12.7" y1="55.88" x2="12.7" y2="48.26" width="0.1524" layer="91"/>
+<pinref part="U$1" gate="U$1" pin="P0.03/AIN1@05"/>
+<wire x1="12.7" y1="48.26" x2="55.88" y2="48.26" width="0.1524" layer="91"/>
 </segment>
 </net>

Commit message: circuit
Parts:
- added C10, C7: 12pF, SparkFun-Capacitors:12PF-0603-50V-5%
- added C5: 0.8pF, SparkFun-Capacitors:0.8PF-0402-50V-0.1PF
- added C6, C9: 100PF, SparkFun-Capacitors:100PF-0402-50V-5%
- added L1: 10uH, Wurth_Automotive_WE-HCFA:WE-HCFA_2818_78436432100
- added L2: 15uH, Wurth_Automotive_WE-MAIA:WE-MAIA_3015_78438335150
- added L4: 3.9nH, Wurth_Signal & Communications_WE-MK:WE-MK_0201_7447820039
- added X1: ABS07-32.768KHZ-T, Crystals_Oscillators:ABS07-32.768KHZ-T
Connections:
- new net N$10: C7.1, U$1.XC2@35, X1.1
- new net N$11: C10.1, U$1.XC1@34, X1.2
- new net N$3: C5.1, L4.1, U$1.ANT@30
- new net N$4: L1.1, U$1.DCC@47
- new net N$5: C6.1, U$1.DEC3@33
- new net N$6: C9.1, U$1.DEC2@32
- new net N$7: L1.2, L2.1
- new net RF: L4.2
- net DEC4: now also L2.2
- net GND: now also C10.2, C5.2, C6.2, C7.2, C9.2, U$1.VSS@31; no longer C3.2
- net N$2: now also C3.2
Other:
- moved on the sheet: C1, C2, C3, C4, C8, POT, U$1

Commit message: reomote circuit
Connections:
- new net N$8: L2.2
- net DEC4: no longer L2.2
Changed lines of the file:
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@@
 <wire x1="33.02" y1="106.68" x2="40.64" y2="106.68" width="0.1524" layer="91"/>
 <wire x1="40.64" y1="106.68" x2="40.64" y2="101.6" width="0.1524" layer="91"/>
-<pinref part="L2" gate="G$1" pin="2"/>
-<wire x1="30.48" y1="111.76" x2="40.64" y2="111.76" width="0.1524" layer="91"/>
-<wire x1="40.64" y1="106.68" x2="40.64" y2="111.76" width="0.1524" layer="91"/>
-<junction x="40.64" y="106.68"/>
 </segment>
 </net>
@@
 </segment>
 </net>
+<net name="N$8" class="0">
+<segment>
+<pinref part="L2" gate="G$1" pin="2"/>
+<wire x1="30.48" y1="111.76" x2="40.64" y2="111.76" width="0.1524" layer="91"/>
+</segment>
+</net>

Commit message: started routing need to add more layers to board
Parts:
- removed C4: 4.7uF, SparkFun-Capacitors:4.7UF-1206-16V-(+80/-20%)
- removed X1: ABS07-32.768KHZ-T, Crystals_Oscillators:ABS07-32.768KHZ-T
- added C11: 4.7uF, SparkFun-Capacitors:4.7UF-0402_TIGHT-6.3V-20%-X5R
- added Y1: ECS-.327-7-38-TR, Crystals_Oscillators:ECS-.327-7-38-TR
- L1: device Wurth_Automotive_WE-HCFA:WE-HCFA_2818_78436432100 -> Wurth_Automotive_WE-MAIA:WE-MAIA_2510_78438323100
Connections:
- net N$1 renamed POTAI
- net N$3 renamed ANT
- net N$4 renamed DCC
- net N$5 renamed DEC3
- net N$6 renamed DEC2
- net N$7 renamed DCC1
- removed net N$10: C7.1, U$1.XC2@35, X1.1
- removed net N$11: C10.1, U$1.XC1@34, X1.2
- removed net N$2: C3.2, U$1.VSS@45
- removed net N$8: L2.2
- new net XC1: C10.1, U$1.XC1@34, Y1.1
- new net XC2: C7.1, U$1.XC2@35, Y1.2
- net DEC4: now also L2.2
- net GND: now also C11.2, C3.2, U$1.VSS@45; no longer C4.2
- net VDD: now also C11.1; no longer C4.1
Other:
- note added: "-Amin Mahjoub"
- note added: "Circuit for the Nordic nRF52832 ble SOC for e-skate remote"
