File: remote_sch.brd (EAGLE design)
At the start: 100 x 80 mm, 16 parts, among them Y1 ECS-.327-7-38-TR

Commit message: stash issue
Routing:
- net XC2: track 19.3 -> 2.19 mm
- net XC1: track 19.1 -> 3.48 mm
- net DEC4: track 14.4 -> 0.00 mm
- net DCC1: track 7.39 -> 0.00 mm
- net DCC: track 8.50 -> 6.08 mm
Changed lines of the file:
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@@
 <attribute name="MANUFACTURER" value="ECS Inc." x="107.95" y="5.08" size="1.778" layer="27" display="off"/>
 <attribute name="MPN" value="ECS-.327-7-38-TR" x="107.95" y="5.08" size="1.778" layer="27" display="off"/>
-<attribute name="NAME" x="55.68593125" y="50.78126875" size="0.61021875" layer="25"/>
 <attribute name="PACKAGE" value="4-SMD" x="107.95" y="5.08" size="1.778" layer="27" display="off"/>
-<attribute name="VALUE" x="55.689859375" y="47.779940625" size="0.609621875" layer="27"/>
 </element>
 <element name="L1" library="Wurth_Automotive_WE-MAIA" library_urn="urn:adsk.eagle:library:14076715" package="WE-MAIA_2510" package3d_urn="urn:adsk.eagle:package:13154127/2" value="10uH" x="33.02" y="52.07" smashed="yes">
@@
 <contactref element="C3" pad="1"/>
 <contactref element="L2" pad="2"/>
-<wire x1="35.43" y1="44.91" x2="35.43" y2="45.72" width="0.1524" layer="1"/>
-<wire x1="39.37" y1="49.53" x2="43.18" y2="49.53" width="0.1524" layer="1"/>
-<wire x1="43.18" y1="49.53" x2="43.18" y2="53.12" width="0.1524" layer="1"/>
-<wire x1="43.18" y1="53.12" x2="42.96" y2="53.34" width="0.1524" layer="1"/>
-<wire x1="35.43" y1="45.72" x2="36.83" y2="47.12" width="0.1524" layer="1"/>
-<wire x1="36.83" y1="47.12" x2="36.83" y2="47.68" width="0.1524" layer="1"/>
-<wire x1="36.83" y1="47.68" x2="37.52" y2="47.68" width="0.1524" layer="1"/>
-<wire x1="37.52" y1="47.68" x2="39.37" y2="49.53" width="0.1524" layer="1"/>
+<wire x1="36.83" y1="47.68" x2="42.96" y2="53.34" width="0" layer="19" extent="1-1"/>
+<wire x1="35.43" y1="44.91" x2="36.83" y2="47.68" width="0" layer="19" extent="1-1"/>
 </signal>
 <signal name="DEC1">
@@
 <contactref element="L1" pad="1"/>
 <wire x1="32.045" y1="50.505" x2="32.045" y2="52.07" width="0.1524" layer="1"/>
-<wire x1="34.9586" y1="44.9814" x2="35.03" y2="44.91" width="0.1524" layer="1"/>
 <wire x1="34.8814" y1="47.1603125" x2="34.8814" y2="47.6686" width="0.1524" layer="1"/>
-<wire x1="35.03" y1="44.91" x2="35.03" y2="47.0117125" width="0.1524" layer="1"/>
-<wire x1="35.03" y1="47.0117125" x2="34.8814" y2="47.1603125" width="0.1524" layer="1"/>
 <wire x1="34.8814" y1="47.6686" x2="32.045" y2="50.505" width="0.1524" layer="1"/>
+<wire x1="35.03" y1="44.91" x2="34.8814" y2="47.1603125" width="0" layer="19" extent="1-1"/>
 </signal>
 <signal name="XC2">
@@
 <contactref element="Y1" pad="4"/>
 <wire x1="39.83" y1="43.71" x2="42.02" y2="43.71" width="0.1524" layer="1"/>
-<wire x1="42.02" y1="43.71" x2="48.26" y2="49.95" width="0.1524" layer="1"/>
-<wire x1="48.26" y1="49.95" x2="56.51" y2="49.95" width="0.1524" layer="1"/>
-<wire x1="56.51" y1="49.95" x2="56.54" y2="49.98" width="0.1524" layer="1"/>
+<wire x1="48.26" y1="49.95" x2="56.54" y2="49.98" width="0" layer="19" extent="1-1"/>
+<wire x1="42.02" y1="43.71" x2="48.26" y2="49.95" width="0" layer="19" extent="1-1"/>
 </signal>
 <signal name="XC1">
@@
 <contactref element="Y1" pad="1"/>
 <wire x1="39.83" y1="43.31" x2="43.31" y2="43.31" width="0.1524" layer="1"/>
-<wire x1="46.14" y1="46.14" x2="49.53" y2="46.14" width="0.1524" layer="1"/>
-<wire x1="43.31" y1="43.31" x2="46.14" y2="46.14" width="0.1524" layer="1"/>
-<wire x1="49.53" y1="46.14" x2="53.6" y2="46.14" width="0.1524" layer="1"/>
-<wire x1="53.6" y1="46.14" x2="56.54" y2="49.08" width="0.1524" layer="1"/>
+<wire x1="49.53" y1="46.14" x2="56.54" y2="49.08" width="0" layer="19" extent="1-1"/>
+<wire x1="43.31" y1="43.31" x2="49.53" y2="46.14" width="0" layer="19" extent="1-1"/>
 </signal>
 <signal name="DCC1">
 <contactref element="L2" pad="1"/>
 <contactref element="L1" pad="2"/>
-<wire x1="40.86" y1="53.34" x2="39.59" y2="52.07" width="0.1524" layer="1"/>
-<wire x1="39.59" y1="52.07" x2="33.995" y2="52.07" width="0.1524" layer="1"/>
+<wire x1="33.995" y1="52.07" x2="40.86" y2="53.34" width="0" layer="19" extent="1-1"/>
 </signal>
 </signals>
